File: hardware/industrial-dual-analog-in-v2.kicad_pcb (KiCad board)
At the start: 2 copper layers, 40 x 40 mm, 81 parts, among them P1 CON-SENSOR2, P2 CONN_1, P3 CONN_8, P4 DEBUG, P5 DEBUG, U1 LMV342IDRG4, U2 LM2664, U3 XMC1100, U4 MCP3911, U5 DRILL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

Commit message: ordered prototype
Other:
- rule pad_to_mask_clearance: 0.2 -> 0
Changed lines of the file:
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@@
   )
   (setup
-    (last_trace_width 0.7)
+    (last_trace_width 0.254)
     (user_trace_width 0.2)
     (user_trace_width 0.25)
@@
     (pad_size 0.45 1.75)
     (pad_drill 0)
-    (pad_to_mask_clearance 0.2)
-    (solder_mask_min_width 0.25)
+    (pad_to_mask_clearance 0)
     (aux_axis_origin 115.6 80)
     (grid_origin 115.6 80)
     (visible_elements FFFFEF3F)
     (pcbplotparams
-      (layerselection 0x00030_80000001)
+      (layerselection 0x010f8_ffffffff)
       (usegerberextensions true)
       (usegerberattributes false)
@@
       (psnegative false)
       (psa4output false)
-      (plotreference true)
-      (plotvalue true)
+      (plotreference false)
+      (plotvalue false)
       (plotinvisibletext false)
       (padsonsilk false)
@@
       (outputformat 1)
       (mirror false)
-      (drillshape 1)
+      (drillshape 0)
       (scaleselection 1)
-      (outputdirectory ""))
+      (outputdirectory "best"))
   )
   (net 0 "")

Commit message: fix logo positions
Parts:
- moved G*** 2.00 mm to (145.6, 100.0)
- moved VAL 2.00 mm to (125.6, 100.0)
Changed lines of the file:
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@@
     (pad_drill 0)
     (pad_to_mask_clearance 0)
+    (solder_mask_min_width 0.25)
     (aux_axis_origin 115.6 80)
     (grid_origin 115.6 80)
@@
   )
   (module kicad-libraries:CE_5mm (layer B.Cu)
-    (at 125.6 102 90)
+    (at 125.6 100 90)
     (fp_text reference VAL (at 0 0 90) (layer B.SilkS) hide
       (effects (font (size 0.2 0.2) (thickness 0.05)) (justify mirror))
@@
   )
   (module kicad-libraries:Logo_CoMCU (layer B.Cu)
-    (at 145.6 102 90)
+    (at 145.6 100 90)
     (fp_text reference G*** (at 0 0 90) (layer B.SilkS) hide
       (effects (font (size 1.524 1.524) (thickness 0.3)) (justify mirror))

Commit message: add detection pin
Connections:
- U3 pad 3: (no net) -> DGND
Routing:
- net DGND: track 62.2 -> 63.2 mm, vias 20 -> 21
Changed lines of the file:
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@@
-(kicad_pcb (version 20171130) (host pcbnew 5.0.2-bee76a0~70~ubuntu18.04.1)
+(kicad_pcb (version 20171130) (host pcbnew 5.1.4-e60b266~84~ubuntu18.04.1)
   (general
     (thickness 1.6)
     (drawings 26)
-    (tracks 688)
+    (tracks 692)
     (zones 0)
     (modules 81)
@@
   )
   (setup
-    (last_trace_width 0.254)
+    (last_trace_width 0.2)
     (user_trace_width 0.2)
     (user_trace_width 0.25)
@@
     (zone_45_only no)
     (trace_min 0.2)
-    (segment_width 0.2)
-    (edge_width 0.15)
     (via_size 0.7)
     (via_drill 0.25)
@@
     (uvia_min_size 0.508)
     (uvia_min_drill 0.127)
+    (edge_width 0.15)
+    (segment_width 0.2)
     (pcb_text_width 0.3)
     (pcb_text_size 1.5 1.5)
@@
     (pad 2 smd oval (at -2.025 -0.75 90) (size 1 0.3) (layers F.Cu F.Paste F.Mask)
       (net 39 "Net-(P4-Pad1)"))
-    (pad 3 smd oval (at -2.025 -0.25 90) (size 1 0.3) (layers F.Cu F.Paste F.Mask))
+    (pad 3 smd oval (at -2.025 -0.25 90) (size 1 0.3) (layers F.Cu F.Paste F.Mask)
+      (net 7 DGND))
     (pad 4 smd oval (at -2.025 0.25 90) (size 1 0.3) (layers F.Cu F.Paste F.Mask))
     (pad 5 smd oval (at -2.025 0.75 90) (size 1 0.3) (layers F.Cu F.Paste F.Mask))
@@
   (segment (start 144.45 88.15) (end 144.6 88.3) (width 0.7) (layer B.Cu) (net 7))
   (via (at 144.6 88.3) (size 0.55) (drill 0.25) (layers F.Cu B.Cu) (net 7))
+  (segment (start 121.46 90.66) (end 121.5 90.7) (width 0.2) (layer F.Cu) (net 7))
+  (via (at 121.5 90.7) (size 0.55) (drill 0.25) (layers F.Cu B.Cu) (net 7))
+  (segment (start 121.46 89.745) (end 121.46 90.66) (width 0.2) (layer F.Cu) (net 7))
   (segment (start 140.7249 90.875) (end 141.2 90.3999) (width 0.254) (layer F.Cu) (net 8))
   (segment (start 138.975 90.875) (end 140.7249 90.875) (width 0.254) (layer F.Cu) (net 8))
@@
   (segment (start 120.2 91.3) (end 119.8 91.3) (width 0.2) (layer F.Cu) (net 39))
   (segment (start 120.96 90.54) (end 120.2 91.3) (width 0.2) (layer F.Cu) (net 39))
-  (segment (start 121.43 92.68) (end 121.43 91.5) (width 0.2) (layer F.Cu) (net 40))
-  (segment (start 123.735 90.145) (end 123.735 88.97) (width 0.2) (layer F.Cu) (net 40))
-  (segment (start 123.23 90.65) (end 123.735 90.145) (width 0.2) (layer F.Cu) (net 40))
   (segment (start 121.43 92.68) (end 121.43 92.28) (width 0.2) (layer F.Cu) (net 40))
-  (segment (start 122.28 90.65) (end 123.23 90.65) (width 0.2) (layer F.Cu) (net 40))
-  (segment (start 121.43 91.5) (end 122.28 90.65) (width 0.2) (layer F.Cu) (net 40))
+  (segment (start 123.735 90.145) (end 123.735 89.32) (width 0.2) (layer F.Cu) (net 40))
+  (segment (start 123.735 89.32) (end 123.735 88.97) (width 0.2) (layer F.Cu) (net 40))
+  (segment (start 123.23 90.65) (end 123.735 90.145) (width 0.2) (layer F.Cu) (net 40))
+  (segment (start 122.327004 90.65) (end 123.23 90.65) (width 0.2) (layer F.Cu) (net 40))
+  (segment (start 121.43 91.547004) (end 122.327004 90.65) (width 0.2) (layer F.Cu) (net 40))
+  (segment (start 121.43 92.68) (end 121.43 91.547004) (width 0.2) (layer F.Cu) (net 40))
   (segment (start 118.97 90.03) (end 117.58 90.03) (width 0.2) (layer F.Cu) (net 41))
   (segment (start 117.345 89.795) (end 117.345 89.4693) (width 0.2) (layer F.Cu) (net 41))
