File: hardware/industrial-dual-analog-in-v2.kicad_pcb (KiCad board)
At the start: 2 copper layers, 40 x 40 mm, 81 parts, among them P1 CON-SENSOR2, P2 CONN_1, P3 CONN_8, P4 DEBUG, P5 DEBUG, U1 LMV342IDRG4, U2 LM2664, U3 XMC1100, U4 MCP3911, U5 DRILL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

Commit message: change opamp type
Parts:
- U1: value LMV342IDRG4 -> TLV272QDRQ1

Commit message: increase version number
Other:
- board text added: "Industrial Dual Analog In 2.2"
- board text removed: "Industrial Dual Analog In 2.1"

Commit message: Data Cleanup
Routing:
- net AGND: track 108.5 -> 106.2 mm
- net Net-(C15-Pad2): track 5.66 -> 4.66 mm
- net Net-(D4-Pad2): track 25.1 -> 24.4 mm
Other:
- net class Default removed
