File: hardware/industrial-dual-analog-in-v2.kicad_sch (KiCad schematic)
At the start: 74 parts

Commit message: fix schematic
Parts:
- C1, C12, C14, C15, C2, C25, C6: value (none) -> 100nF; footprint (none) -> kicad-libraries:C0603F
- C10, C11: value (none) -> 1nF; footprint (none) -> kicad-libraries:C0603F
- C13, C16: value (none) -> 10µF; footprint (none) -> kicad-libraries:C0603F
- C17, C19, C20, C22: value (none) -> 15pF; footprint (none) -> kicad-libraries:C0603F
- C18, C21: value (none) -> 150pF; footprint (none) -> kicad-libraries:C0603F
- C23: value (none) -> 220pF; footprint (none) -> kicad-libraries:C0402F
- C24: value (none) -> 1uF; footprint (none) -> kicad-libraries:C0603F
- C3, C4, C5: value (none) -> 3.3µF; footprint (none) -> kicad-libraries:C0603F
- C7: value (none) -> 10uF; footprint (none) -> kicad-libraries:C0805
- C8, C9: value (none) -> 18pF; footprint (none) -> kicad-libraries:C0603F
- D1: value (none) -> CDSOD323-T05SC; footprint (none) -> kicad-libraries:SOD-323
- D2: value (none) -> CDSOD323-T03SC; footprint (none) -> kicad-libraries:SOD-323
- D3, D4, D5: value (none) -> blue; footprint (none) -> kicad-libraries:D0603F
- F1, F2: value (none) -> OZCJ0035FF2G; footprint (none) -> kicad-libraries:F1206
- FB1, FB2: value (none) -> FILTER; footprint (none) -> kicad-libraries:C0603F
- P1: value (none) -> CON-SENSOR2; footprint (none) -> kicad-libraries:CON-SENSOR2
- P2: value (none) -> CONN_1; footprint (none) -> kicad-libraries:PINTST
- P3: value (none) -> CONN_8; footprint (none) -> kicad-libraries:OQ_8P
- P4: value (none) -> DEBUG; footprint (none) -> kicad-libraries:DEBUG_PAD
- P5: value (none) -> DEBUG; footprint (none) -> kicad-libraries:SolderJumper
- R1: value (none) -> 0; footprint (none) -> kicad-libraries:R0603F
- R10, R11, R8, R9: value (none) -> 4k7/10ppm; footprint (none) -> kicad-libraries:R0603F
- R12, R17, R18, R19, R20, R7: value (none) -> 10; footprint (none) -> kicad-libraries:R0603F
- R13, R14, R15, R16: value (none) -> 280k/10ppm; footprint (none) -> kicad-libraries:R0603F
- R2: value (none) -> 1M; footprint (none) -> kicad-libraries:R0603F
- R21, R22, R23, R24, R3: value (none) -> 100k; footprint (none) -> kicad-libraries:R0603F
- R5, R6: value (none) -> 68.1; footprint (none) -> kicad-libraries:R0603F
- RP1, RP2: value (none) -> 82; footprint (none) -> kicad-libraries:4X0402
- RP3: value (none) -> 1k; footprint (none) -> kicad-libraries:4X0402
- U1: value (none) -> TLV272QDRQ1; footprint (none) -> kicad-libraries:SOIC8
- U2: value (none) -> LM2664; footprint (none) -> kicad-libraries:SOT23-6
- U3: value (none) -> XMC1100; footprint (none) -> kicad-libraries:QFN24-4x4mm-0.5mm
- U4: value (none) -> MCP3911; footprint (none) -> kicad-libraries:SSOP20-53
- U5, U6, U7, U8: value (none) -> DRILL; footprint (none) -> kicad-libraries:DRILL_NP
- X1: value (none) -> 4MHz; footprint (none) -> kicad-libraries:HC49_US
